Commit message: 'Added sending movp commands over modbus'

File: arm_description/urdf/delta_urdf_v2.urdf (robot description, URDF)
Before this commit: robot delta_urdf_v2, 7 links, 6 joints
Joints:
- joint wrist3: limit lower=-2.0943951024 upper=2.0943951024 effort=9.5120444234 velocity=7 -> lower=2.0943951024 upper=-2.0943951024 effort=9.5120444234 velocity=7

Commit message: URDF model fixes

File: arm_description/urdf/delta_urdf_v2.urdf (robot description, URDF)
Before this commit: robot delta_urdf_v2, 7 links, 6 joints
Links:
- added link base
Joints:
- added joint dummy_joint: type fixed, parent base_link, child base, origin xyz=0 0 0 rpy=1.57079632679 0 0, axis 0 0 1
- joint wrist2: origin xyz=0.0400000444661043 -0.435000000020256 0 rpy=-3.14159265358979 0 1.5707963267949 -> xyz=0.0400000444661043 0.435000000020256 0 rpy=0 0 -1.5707963267949

Commit message: Fixed base frame

File: arm_description/urdf/delta_urdf_v2.urdf (robot description, URDF)
Before this commit: robot delta_urdf_v2, 8 links, 7 joints
Joints:
- joint dummy_joint: origin xyz=0 0 0 rpy=1.57079632679 0 0 -> xyz=0 0 0 rpy=1.57079632679 -1.57079632679 0

Commit message: Fixed wrist joint

File: arm_description/urdf/delta_urdf_v2.urdf (robot description, URDF)
Before this commit: robot delta_urdf_v2, 8 links, 7 joints
Joints:
- joint wrist3: origin xyz=0.0330000000202569 0 0 rpy=1.5707963267949 0 1.5707963267949 -> xyz=0 0.0330000000202569 0 rpy=1.5707963267949 0 1.5707963267949
