Commit message: Added end effector to URDF model

File: arm_description/urdf/arm_with_endeffector.urdf.xacro (robot description, xacro)
@@ -1,7 +1,7 @@
 <robot name="myrobot" xmlns:xacro="http://www.ros.org/wiki/xacro" xmlns:xi="http://www.w3.org/2001/XInclude">
 <xacro:include filename="$(find arm_description)/urdf/delta_urdf_v2.urdf"/>
-<xacro:include filename="$(find arm_description)/urdf/robotiq_ft300.urdf.xacro" />
-    <xacro:robotiq_ft300 parent="wrist4_link" prefix="ft300/">
+<xacro:include filename="$(find arm_description)/urdf/end_effector.urdf.xacro" />
+    <xacro:end_effector parent="wrist4_link" prefix="EE/">
         <origin xyz="0 0 0" rpy="0 -1.57079632679489661923 0"/>
-    </xacro:robotiq_ft300>
+    </xacro:end_effector>
 </robot>

File: arm_description/urdf/delta_urdf_v2.urdf (robot description, URDF)
Before this commit: robot delta_urdf_v2, 8 links, 7 joints
Joints:
- joint wrist3: origin xyz=0 0.0330000000202569 0 rpy=1.5707963267949 0 1.5707963267949 -> xyz=0.0330000000202569 0 0 rpy=1.5707963267949 0 1.5707963267949
